Commit message: URDF标准化：STL后缀改为小写stl；关节名称中-改为_；XML标签行合并为单行
- STL文件后缀：.STL -> .stl（28个文件重命名）
- 关节命名：J1-1 -> J1_1（URDF、nova.yaml、arm_control.py统一修改）
- XML标签：所有多行标签合并为单行（origin, mass, inertia, mesh, material等）
- 文件优化：URDF从2229行减少到1401行
- 配置文件同步：nova.yaml关节列表、arm_control.py关节名称同步更新

File: simulation/src/nova_sim/urdf/nova_robot.urdf (robot description, URDF)
Before this commit: robot nova_robot, 40 links, 39 joints
Links:
- removed link J1-1
- removed link J1-2
- removed link J1-3
- removed link J1-4
- removed link J1-5
- removed link J1-6
- removed link J1-7
- removed link J1-8
- removed link J2-1
- removed link J2-2
- removed link J2-3
- removed link J2-4
- removed link J2-5
- removed link J2-6
- removed link J2-7
- removed link J2-8
- removed link J3-1
- removed link J3-2
- removed link J3-3
- removed link J3-4
- removed link J3-5
- removed link J3-6
- removed link J4-1
- removed link J4-2
- removed link J4-3
- removed link J4-4
- removed link J4-5
- removed link J4-6
- added link J1_1, mass 0.803381596273923; collision mesh filename=package://nova_sim/meshes/J1_1.stl; visual mesh filename=package://nova_sim/meshes/J1_1.stl
- added link J1_2, mass 1.57815566164452; collision mesh filename=package://nova_sim/meshes/J1_2.stl; visual mesh filename=package://nova_sim/meshes/J1_2.stl
- added link J1_3, mass 0.999485676814869; collision mesh filename=package://nova_sim/meshes/J1_3.stl; visual mesh filename=package://nova_sim/meshes/J1_3.stl
- added link J1_4, mass 0.441710014889936; collision mesh filename=package://nova_sim/meshes/J1_4.stl; visual mesh filename=package://nova_sim/meshes/J1_4.stl
- added link J1_5, mass 0.585231261599067; collision mesh filename=package://nova_sim/meshes/J1_5.stl; visual mesh filename=package://nova_sim/meshes/J1_5.stl
- added link J1_6, mass 0.328138288054857; collision mesh filename=package://nova_sim/meshes/J1_6.stl; visual mesh filename=package://nova_sim/meshes/J1_6.stl
- added link J1_7, mass 0.0552137973288012; collision mesh filename=package://nova_sim/meshes/J1_7.stl; visual mesh filename=package://nova_sim/meshes/J1_7.stl
- added link J1_8, mass 0.0552137973963911; collision mesh filename=package://nova_sim/meshes/J1_8.stl; visual mesh filename=package://nova_sim/meshes/J1_8.stl
- added link J2_1, mass 0.80338159626503; collision mesh filename=package://nova_sim/meshes/J2_1.stl; visual mesh filename=package://nova_sim/meshes/J2_1.stl
- added link J2_2, mass 1.5781557465293; collision mesh filename=package://nova_sim/meshes/J2_2.stl; visual mesh filename=package://nova_sim/meshes/J2_2.stl
- added link J2_3, mass 0.999485676814903; collision mesh filename=package://nova_sim/meshes/J2_3.stl; visual mesh filename=package://nova_sim/meshes/J2_3.stl
- added link J2_4, mass 0.441710147759153; collision mesh filename=package://nova_sim/meshes/J2_4.stl; visual mesh filename=package://nova_sim/meshes/J2_4.stl
- added link J2_5, mass 0.585231256875491; collision mesh filename=package://nova_sim/meshes/J2_5.stl; visual mesh filename=package://nova_sim/meshes/J2_5.stl
- added link J2_6, mass 0.328138288054906; collision mesh filename=package://nova_sim/meshes/J2_6.stl; visual mesh filename=package://nova_sim/meshes/J2_6.stl
- added link J2_7, mass 0.0552137973963913; collision mesh filename=package://nova_sim/meshes/J2_7.stl; visual mesh filename=package://nova_sim/meshes/J2_7.stl
- added link J2_8, mass 0.0552137973288004; collision mesh filename=package://nova_sim/meshes/J2_8.stl; visual mesh filename=package://nova_sim/meshes/J2_8.stl
- added link J3_1, mass 0.130770244382924; collision mesh filename=package://nova_sim/meshes/J3_1.stl; visual mesh filename=package://nova_sim/meshes/J3_1.stl
- added link J3_2, mass 0.0832278336056144; collision mesh filename=package://nova_sim/meshes/J3_2.stl; visual mesh filename=package://nova_sim/meshes/J3_2.stl
- added link J3_3, mass 0.0569984713380656; collision mesh filename=package://nova_sim/meshes/J3_3.stl; visual mesh filename=package://nova_sim/meshes/J3_3.stl
- added link J3_4, mass 0.034634178423434; collision mesh filename=package://nova_sim/meshes/J3_4.stl; visual mesh filename=package://nova_sim/meshes/J3_4.stl
- added link J3_5, mass 0.0356972566661433; collision mesh filename=package://nova_sim/meshes/J3_5.stl; visual mesh filename=package://nova_sim/meshes/J3_5.stl
- added link J3_6, mass 0.0650882430291389; collision mesh filename=package://nova_sim/meshes/J3_6.stl; visual mesh filename=package://nova_sim/meshes/J3_6.stl
- added link J4_1, mass 0.130770244383303; collision mesh filename=package://nova_sim/meshes/J4_1.stl; visual mesh filename=package://nova_sim/meshes/J4_1.stl
- added link J4_2, mass 0.0832278323735664; collision mesh filename=package://nova_sim/meshes/J4_2.stl; visual mesh filename=package://nova_sim/meshes/J4_2.stl
- added link J4_3, mass 0.0569984708957405; collision mesh filename=package://nova_sim/meshes/J4_3.stl; visual mesh filename=package://nova_sim/meshes/J4_3.stl
- added link J4_4, mass 0.0346341792586891; collision mesh filename=package://nova_sim/meshes/J4_4.stl; visual mesh filename=package://nova_sim/meshes/J4_4.stl
- added link J4_5, mass 0.0356972565577711; collision mesh filename=package://nova_sim/meshes/J4_5.stl; visual mesh filename=package://nova_sim/meshes/J4_5.stl
- added link J4_6, mass 0.0650882038377387; collision mesh filename=package://nova_sim/meshes/J4_6.stl; visual mesh filename=package://nova_sim/meshes/J4_6.stl
Joints:
- removed joint J1-1_joint
- removed joint J1-2_joint
- removed joint J1-3_joint
- removed joint J1-4_joint
- removed joint J1-5_joint
- removed joint J1-6_joint
- removed joint J1-7_joint
- removed joint J1-8_joint
- removed joint J2-1_joint
- removed joint J2-2_joint
- removed joint J2-3_joint
- removed joint J2-4_joint
- removed joint J2-5_joint
- removed joint J2-6_joint
- removed joint J2-7_joint
- removed joint J2-8_joint
- removed joint J3-1_joint
- removed joint J3-2_joint
- removed joint J3-3_joint
- removed joint J3-4_joint
- removed joint J3-5_joint
- removed joint J3-6_joint
- removed joint J4-1_joint
- removed joint J4-2_joint
- removed joint J4-3_joint
- removed joint J4-4_joint
- removed joint J4-5_joint
- removed joint J4-6_joint
- added joint J1_1_joint: type revolute, parent base_link, child J1_1, origin xyz=0 0 0.2234 rpy=0 0 0, axis 0 0 -1, limit lower=-3.14 upper=3.14 effort=100 velocity=2
- added joint J1_2_joint: type revolute, parent J1_1, child J1_2, origin xyz=0 0 0 rpy=-1.5708 0 3.1416, axis 0 0 1, limit lower=-3.14 upper=3.14 effort=100 velocity=2
- added joint J1_3_joint: type revolute, parent J1_2, child J1_3, origin xyz=0 -0.28 0 rpy=0 0 1.5708, axis 0 0 -1, limit lower=-3.14 upper=3.14 effort=100 velocity=2
- added joint J1_4_joint: type revolute, parent J1_3, child J1_4, origin xyz=0 0.225 0.1175 rpy=3.1416 0 0, axis 0 0 1, limit lower=-3.14 upper=3.14 effort=100 velocity=2
- added joint J1_5_joint: type revolute, parent J1_4, child J1_5, origin xyz=0 -0.12 0 rpy=1.5708 1.5708 0, axis 0 0 1, limit lower=-3.14 upper=3.14 effort=100 velocity=2
- added joint J1_6_joint: type revolute, parent J1_5, child J1_6, origin xyz=0 0.087743 0 rpy=-1.5708 0 0, axis 0 0 1, limit lower=-3.14 upper=3.14 effort=100 velocity=2
- added joint J1_7_joint: type prismatic, parent J1_6, child J1_7, origin xyz=-0.0625 -0.024005 0.11568 rpy=1.5708 0 1.5708, axis 0 0 -1, limit lower=-0.1 upper=0.1 effort=100 velocity=2
- added joint J1_8_joint: type prismatic, parent J1_6, child J1_8, origin xyz=0.0625 -0.024005 0.11568 rpy=-1.5708 0 1.5708, axis 0 0 1, limit lower=-3.14 upper=3.14 effort=100 velocity=2
- added joint J2_1_joint: type revolute, parent base_link, child J2_1, origin xyz=1.06 0 0.2234 rpy=0 0 0, axis 0 0 1, limit lower=-3.14 upper=3.14 effort=100 velocity=2
- added joint J2_2_joint: type revolute, parent J2_1, child J2_2, origin xyz=0 0 0 rpy=-1.5708 0 3.1416, axis 0 0 1, limit lower=-3.14 upper=3.14 effort=100 velocity=2
- added joint J2_3_joint: type revolute, parent J2_2, child J2_3, origin xyz=0 -0.28 0 rpy=0 0 0, axis 0 0 1, limit lower=-3.14 upper=3.14 effort=100 velocity=2
- added joint J2_4_joint: type revolute, parent J2_3, child J2_4, origin xyz=0.225 0 0.1175 rpy=3.1416 0 3.1416, axis 0 0 1, limit lower=-3.14 upper=3.14 effort=100 velocity=2
- added joint J2_5_joint: type revolute, parent J2_4, child J2_5, origin xyz=-0.12 0 0 rpy=1.5708 0 -1.5708, axis 0 0 -1, limit lower=-3.14 upper=3.14 effort=100 velocity=2
- added joint J2_6_joint: type revolute, parent J2_5, child J2_6, origin xyz=-0.087743 0 0 rpy=-1.5708 0 1.5708, axis 0 0 1, limit lower=-3.14 upper=3.14 effort=100 velocity=2
- added joint J2_7_joint: type prismatic, parent J2_6, child J2_7, origin xyz=0.0625 0.023995 0.11568 rpy=1.5708 0 -1.5708, axis 0 0 -1, limit lower=-0.1 upper=0.1 effort=100 velocity=2
- added joint J2_8_joint: type prismatic, parent J2_6, child J2_8, origin xyz=-0.0625 0.023995 0.11568 rpy=-1.5708 0 -1.5708, axis 0 0 1, limit lower=-0.1 upper=0.1 effort=100 velocity=2
- added joint J3_1_joint: type revolute, parent base_link, child J3_1, origin xyz=0.2 -0.575 0.15855 rpy=0 0 3.1416, axis 0 0 1, limit lower=-3.14 upper=3.14 effort=100 velocity=2
- added joint J3_2_joint: type revolute, parent J3_1, child J3_2, origin xyz=0 0 0 rpy=-1.5708 0 0, axis 0 0 1, limit lower=-3.14 upper=3.14 effort=100 velocity=2
- added joint J3_3_joint: type revolute, parent J3_2, child J3_3, origin xyz=0.0005 -0.19575 0.0275 rpy=3.1416 0 3.1416, axis 0 0 -1, limit lower=-3.14 upper=3.14 effort=100 velocity=2
- added joint J3_4_joint: type revolute, parent J3_3, child J3_4, origin xyz=0.1537 0.0011225 -0.002 rpy=0 0 3.1416, axis 0 0 -1, limit lower=-3.14 upper=3.14 effort=100 velocity=2
- added joint J3_5_joint: type revolute, parent J3_4, child J3_5, origin xyz=0.0019999 1.4606E-05 -0.05345 rpy=-1.5708 0 -1.5635, axis 0 0 -1, limit lower=-3.14 upper=3.14 effort=100 velocity=2
- added joint J3_6_joint: type revolute, parent J3_5, child J3_6, origin xyz=0 0.031 -0.08645 rpy=1.5708 -1.5635 0, axis 0 0 -1, limit lower=-3.14 upper=3.14 effort=100 velocity=2
- added joint J4_1_joint: type revolute, parent base_link, child J4_1, origin xyz=0.86 -0.575 0.15855 rpy=0 0 0, axis 0 0 1, limit lower=-3.14 upper=3.14 effort=100 velocity=2
- added joint J4_2_joint: type revolute, parent J4_1, child J4_2, origin xyz=0 0 0 rpy=-1.5708 0 3.1416, axis 0 0 1, limit lower=-3.14 upper=3.14 effort=100 velocity=2
- added joint J4_3_joint: type revolute, parent J4_2, child J4_3, origin xyz=0 -0.19575 0.0275 rpy=3.1416 0 3.1416, axis 0 0 -1, limit lower=-3.14 upper=3.14 effort=100 velocity=2
- added joint J4_4_joint: type revolute, parent J4_3, child J4_4, origin xyz=-0.15369 0.0018579 -0.002 rpy=0 0 3.1416, axis 0 0 -1, limit lower=-3.14 upper=3.14 effort=100 velocity=2
- added joint J4_5_joint: type revolute, parent J4_4, child J4_5, origin xyz=-0.0019999 2.4176E-05 -0.05375 rpy=1.5708 0 -1.5829, axis 0 0 -1, limit lower=-3.14 upper=3.14 effort=100 velocity=2
- added joint J4_6_joint: type revolute, parent J4_5, child J4_6, origin xyz=0 -0.031 -0.08645 rpy=1.5708 1.5587 3.1416, axis 0 0 -1, limit lower=-3.14 upper=3.14 effort=100 velocity=2
- joint camera1_joint: parent J1-6 -> J1_6
- joint camera2_joint: parent J2-6 -> J2_6

Commit message: nova_sim: sync simulation tuning and visual config from nova_test

File: simulation/src/nova_sim/urdf/nova_robot.urdf (robot description, URDF)
Before this commit: robot nova_robot, 40 links, 39 joints
Links:
- removed link world
Joints:
- removed joint world_to_base
- joint camera0_joint: origin xyz=0 0 -0.15 rpy=1.57 2.24 0 -> xyz=0 0 -0.15 rpy=1.57 2.24 1.5708
- joint camera0_optical_joint: origin xyz=0 0 0 rpy=-1.57079632679 0 -1.57079632679 -> xyz=0 0 0 rpy=-1.57079632679 0 0
- joint camera1_joint: origin xyz=0 -0.08 0.041 rpy=0 -1.57 0 -> xyz=0 -0.08 0.041 rpy=0 -1.57 1.5708
- joint camera1_optical_joint: origin xyz=0 0 0 rpy=-1.57079632679 0 -1.57079632679 -> xyz=0 0 0 rpy=-1.57079632679 0 0
- joint camera2_joint: origin xyz=0 -0.08 0.041 rpy=0 -1.57 0 -> xyz=0 -0.08 0.041 rpy=0 -1.57 1.5708
- joint camera2_optical_joint: origin xyz=0 0 0 rpy=-1.57079632679 0 -1.57079632679 -> xyz=0 0 0 rpy=-1.57079632679 0 0

File: simulation/src/nova_sim/urdf/nova_robot_position.urdf (robot description, URDF)
Before this commit: robot nova_robot, 40 links, 39 joints
Links:
- removed link world
Joints:
- removed joint world_to_base
- joint camera0_joint: origin xyz=0 0 -0.15 rpy=1.57 2.24 0 -> xyz=0 0 -0.15 rpy=1.57 1.57 -1.5708
- joint camera0_optical_joint: origin xyz=0 0 0 rpy=-1.57079632679 0 -1.57079632679 -> xyz=0 0 0 rpy=-1.57079632679 0 0
- joint camera1_joint: origin xyz=0 -0.08 0.041 rpy=0 -1.57 0 -> xyz=0 -0.08 0.041 rpy=0 -1.57 1.5708
- joint camera1_optical_joint: origin xyz=0 0 0 rpy=-1.57079632679 0 -1.57079632679 -> xyz=0 0 0 rpy=-1.57079632679 0 0
- joint camera2_joint: origin xyz=0 -0.08 0.041 rpy=0 -1.57 0 -> xyz=0 -0.08 0.041 rpy=0 -1.57 1.5708
- joint camera2_optical_joint: origin xyz=0 0 0 rpy=-1.57079632679 0 -1.57079632679 -> xyz=0 0 0 rpy=-1.57079632679 0 0
