Commit message: fix: correct J1_8_joint prismatic limit and urdf default path

File: simulation/src/nova_sim/urdf/nova_robot_position.urdf (robot description, URDF)
Before this commit: robot nova_robot, 40 links, 39 joints
Joints:
- joint J1_8_joint: limit lower=-3.14 upper=3.14 effort=100 velocity=2 -> lower=-0.1 upper=0.1 effort=100 velocity=2

Commit message: nova_sim: sync MoveIt2 and Qt control workflow
Migrate the latest MoveIt2 executor and Qt control UI updates into nova_sim, including pose/joint interaction improvements and launch integration for current simulation testing.

Made-with: Cursor

File: simulation/src/nova_sim/urdf/nova_robot_position.urdf (robot description, URDF)
Before this commit: robot nova_robot, 39 links, 38 joints
Joints:
- joint J1_7_joint: limit lower=-0.1 upper=0.1 effort=100 velocity=2 -> lower=-0.04 upper=0.02 effort=100 velocity=2
- joint J1_8_joint: limit lower=-0.1 upper=0.1 effort=100 velocity=2 -> lower=-0.02 upper=0.04 effort=100 velocity=2
- joint J2_7_joint: limit lower=-0.1 upper=0.1 effort=100 velocity=2 -> lower=-0.04 upper=0.02 effort=100 velocity=2
- joint J2_8_joint: limit lower=-0.1 upper=0.1 effort=100 velocity=2 -> lower=-0.02 upper=0.04 effort=100 velocity=2

Commit message: nova_sim: sync with nova_test collision, control and D405 camera tuning

File: simulation/src/nova_sim/urdf/nova_robot_position.urdf (robot description, URDF)
Before this commit: robot nova_robot, 39 links, 38 joints
Links:
- link base_link: geometry collision box size=1.40 0.96 0.03; visual mesh filename=package://nova_sim/meshes/base_link.stl
