Commit message: nova_sim: sync camera, aruco, and spawn pipeline updates
Align nova_sim with the validated nova_test setup by switching to xacro-based spawning, fixing optical frame orientation and depth ranges, and adding dual aruco board mounting with UV-mapped board mesh support.

Made-with: Cursor

File: simulation/src/nova_sim/urdf/aruco_cali.xacro (robot description, xacro)
@@ -8,5 +8,5 @@
     <xacro:property name="board_thickness" value="0.001"/>
     <!-- 连接到父链接的关节 -->
-    <joint name="base_to_aruco_joint" type="fixed">
+    <joint name="${child_link}_joint" type="fixed">
       <origin xyz="${cali_x} ${cali_y} ${cali_z}"
               rpy="${cali_roll} ${cali_pitch} ${cali_yaw}"/>
@@ -19,9 +19,7 @@
         <origin xyz="0 0 0" rpy="0 0 0"/>
         <geometry>
-          <box size="${board_width} ${board_height} ${board_thickness}"/>
+          <!-- 使用带UV的平面网格贴图，Gazebo 对这种方式兼容性更好 -->
+          <mesh filename="package://nova_sim/meshes/aruco_board.dae"/>
         </geometry>
-        <material name="aruco_texture">
-          <texture filename="package://nova_sim/meshes/6x6_1000-0.png"/>
-        </material>
       </visual>
       <collision>
@@ -37,19 +35,14 @@
       </inertial>
     </link>
-    <!-- Gazebo 配置 - 使用纹理贴图 -->
+    <!-- Gazebo 配置 -->
     <gazebo reference="${child_link}">
       <mu1>0.5</mu1>
       <mu2>0.5</mu2>
-      <visual>
-        <material>
-          <diffuse>1 1 1 1</diffuse>
-          <specular>0 0 0 0</specular>
-          <pbr>
-            <metal>
-              <albedo_map>package://nova_sim/meshes/6x6_1000-0.png</albedo_map>
-            </metal>
-          </pbr>
-        </material>
-      </visual>
+      <material>
+        <ambient>1 1 1 1</ambient>
+        <diffuse>1 1 1 1</diffuse>
+        <specular>0 0 0 1</specular>
+        <emissive>0 0 0 1</emissive>
+      </material>
     </gazebo>
     <!-- ArUco 标记可视化（使用白色板子，实际识别由视觉系统处理） -->

File: simulation/src/nova_sim/urdf/nova_robot.urdf (robot description, URDF)
Before this commit: robot nova_robot, 39 links, 38 joints
Joints:
- joint camera0_optical_joint: origin xyz=0 0 0 rpy=-1.57079632679 0 0 -> xyz=0 0 0 rpy=-1.57079632679 0 -1.57079632679
- joint camera1_optical_joint: origin xyz=0 0 0 rpy=-1.57079632679 0 0 -> xyz=0 0 0 rpy=-1.57079632679 0 -1.57079632679
- joint camera2_optical_joint: origin xyz=0 0 0 rpy=-1.57079632679 0 0 -> xyz=0 0 0 rpy=-1.57079632679 0 -1.57079632679

File: simulation/src/nova_sim/urdf/nova_robot_position.urdf (robot description, URDF)
Before this commit: robot nova_robot, 39 links, 38 joints
Joints:
- joint camera0_optical_joint: origin xyz=0 0 0 rpy=-1.57079632679 0 0 -> xyz=0 0 0 rpy=-1.57079632679 0 -1.57079632679
- joint camera1_optical_joint: origin xyz=0 0 0 rpy=-1.57079632679 0 0 -> xyz=0 0 0 rpy=-1.57079632679 0 -1.57079632679
- joint camera2_optical_joint: origin xyz=0 0 0 rpy=-1.57079632679 0 0 -> xyz=0 0 0 rpy=-1.57079632679 0 -1.57079632679

Commit message: calib_sim: integrate Qt workflow and stabilize calibration pipeline
Merge the ROS2 Qt calibration UI and sample export flow, and tune detection/solver behavior with improved simulation rendering settings in nova_sim for more consistent calibration runs.

Made-with: Cursor

File: simulation/src/nova_sim/urdf/aruco_cali.xacro (robot description, xacro)
@@ -2,5 +2,5 @@
 <robot xmlns:xacro="http://www.ros.org/wiki/xacro" name="aruco_cali">
   <!-- 定义 aruco_cali 宏 -->
-  <xacro:macro name="aruco_cali" params="parent_link child_link cali_x cali_y cali_z cali_roll cali_pitch cali_yaw">
+  <xacro:macro name="aruco_cali" params="parent_link child_link cali_x cali_y cali_z cali_roll cali_pitch cali_yaw mesh_file:='package://nova_sim/meshes/aruco_board.dae'">
     <!-- ArUco 标定板尺寸参数 -->
     <xacro:property name="board_width" value="0.1"/>
@@ -20,5 +20,5 @@
         <geometry>
           <!-- 使用带UV的平面网格贴图，Gazebo 对这种方式兼容性更好 -->
-          <mesh filename="package://nova_sim/meshes/aruco_board.dae"/>
+          <mesh filename="${mesh_file}"/>
         </geometry>
       </visual>
