Commit message: feat(nova_sim_mujoco): MuJoCo 正常启动 Nova 并显示四块 ArUco 标定板
- MJCF 转换保留标定板；薄盒 DAE 满足网格体积，避免 inertia 报错
- 四块板 DICT_6X6_1000 id0–3 命名与纹理；6x6_1000-2.png 白边与其它一致
- 顶/底面 UV 与 scripts/regenerate_aruco_board_daes.py 可再生
- calib_sim_mujoco 眼在手上 target_marker 与底座板 id 对齐
- 移除未用 USD/svg/base_link.dae；simulation Cursor 规则仅改 mujoco 分包

Made-with: Cursor

File: simulation/src/nova_sim_mujoco/urdf/aruco_cali.xacro (robot description, xacro)
@@ -2,5 +2,5 @@
 <robot xmlns:xacro="http://www.ros.org/wiki/xacro" name="aruco_cali">
   <!-- 定义 aruco_cali 宏 -->
-  <xacro:macro name="aruco_cali" params="parent_link child_link cali_x cali_y cali_z cali_roll cali_pitch cali_yaw mesh_file:='package://nova_sim/meshes/aruco_board.dae'">
+  <xacro:macro name="aruco_cali" params="parent_link child_link cali_x cali_y cali_z cali_roll cali_pitch cali_yaw mesh_file:='package://nova_sim/meshes/aruco_6x6_1000_id0.dae'">
     <!-- ArUco 标定板尺寸参数 -->
     <xacro:property name="board_width" value="0.1"/>
@@ -17,5 +17,5 @@
     <link name="${child_link}">
       <visual>
-        <!-- 翻面已在 aruco_board*.dae 内用法线/绕序完成；此处勿再 rpy 转 180°，否则易镜像。 -->
+        <!-- 翻面已在 aruco_6x6_1000_id*.dae 内用法线/绕序完成；此处勿再 rpy 转 180°，否则易镜像。 -->
         <origin xyz="0 0 0" rpy="0 0 0"/>
         <geometry>
