Commit message: simulation(calib_sim_mujoco,nova_sim_mujoco): stabilize eye-in-hand calibration pipeline
Align MuJoCo camera mounting/orientation and calibration sampling defaults so eih workflows produce stable, usable results with consistent topics, marker mapping, and mirror-safe ArUco pose estimation.

Made-with: Cursor

File: simulation/src/nova_sim_mujoco/urdf/nova_robot_position.urdf (robot description, URDF)
Before this commit: robot nova_robot, 39 links, 38 joints
Links:
- added link camera0_frustum; visual cylinder length=0.30 radius=0.06
- added link camera1_frustum; visual cylinder length=0.30 radius=0.06
- added link camera2_frustum; visual cylinder length=0.30 radius=0.06
Joints:
- added joint camera0_frustum_joint: type fixed, parent camera0_optical_frame, child camera0_frustum, origin xyz=0 0 0 rpy=0 0 0
- added joint camera1_frustum_joint: type fixed, parent camera1_optical_frame, child camera1_frustum, origin xyz=0 0 0 rpy=0 0 0
- added joint camera2_frustum_joint: type fixed, parent camera2_optical_frame, child camera2_frustum, origin xyz=0 0 0 rpy=0 0 0
