Commit message: fix(gazebo_robot_had2503_demo): stabilize physics and raise chassis speed limits
Use AABB/cylinder collisions instead of dense STL meshes to stop ODE fly-away
and OOM kills; soften world contacts and raise debug UI / diff_drive cmd_vel limits.

Co-authored-by: Cursor <cursoragent@cursor.com>

File: simulation/src/gazebo_robot_had2503_demo/urdf/had2503.gazebo.xacro (robot description, xacro)
@@ -1,17 +1,78 @@
 <?xml version="1.0"?>
 <robot xmlns:xacro="http://www.ros.org/wiki/xacro" name="HAD2503-D-DEX1">
-  <!-- xacro 会扁平化嵌套的 <robot> include -->
+  <!-- 视觉仍为 STL；碰撞已在 had2503_links 中改为 AABB，避免 ODE 飞车/OOM -->
   <xacro:include filename="$(find gazebo_robot_had2503_demo)/urdf/had2503_links.urdf.xacro"/>
+  <!-- 关闭自碰；驱动轮摩擦 -->
+  <xacro:macro name="link_gazebo" params="link">
+    <gazebo reference="${link}">
+      <selfCollide>false</selfCollide>
+    </gazebo>
+  </xacro:macro>
+  <xacro:link_gazebo link="base_link"/>
+  <xacro:link_gazebo link="ankle_pitch_link"/>
+  <xacro:link_gazebo link="knee_pitch_link"/>
+  <xacro:link_gazebo link="hip_pitch_link"/>
+  <xacro:link_gazebo link="waist_yaw_link"/>
+  <xacro:link_gazebo link="waist_pitch_link"/>
+  <xacro:link_gazebo link="waist_roll_link"/>
+  <xacro:link_gazebo link="head_yaw_link"/>
+  <xacro:link_gazebo link="head_pitch_link"/>
+  <xacro:link_gazebo link="left_shoulder_pitch_link"/>
+  <xacro:link_gazebo link="left_shoulder_roll_link"/>
+  <xacro:link_gazebo link="left_shoulder_yaw_link"/>
+  <xacro:link_gazebo link="left_elbow_link"/>
+  <xacro:link_gazebo link="left_wrist_yaw_link"/>
+  <xacro:link_gazebo link="left_wrist_pitch_link"/>
+  <xacro:link_gazebo link="left_wrist_roll_link"/>
+  <xacro:link_gazebo link="right_shoulder_pitch_link"/>
+  <xacro:link_gazebo link="right_shoulder_roll_link"/>
+  <xacro:link_gazebo link="right_shoulder_yaw_link"/>
+  <xacro:link_gazebo link="right_elbow_link"/>
+  <xacro:link_gazebo link="right_wrist_yaw_link"/>
+  <xacro:link_gazebo link="right_wrist_pitch_link"/>
+  <xacro:link_gazebo link="right_wrist_roll_link"/>
   <gazebo reference="left_wheel_link">
-    <mu1>1.0</mu1>
-    <mu2>1.0</mu2>
-    <kp>1e5</kp>
-    <kd>1.0</kd>
+    <selfCollide>false</selfCollide>
+    <mu1>1.2</mu1>
+    <mu2>1.2</mu2>
+    <kp>1e4</kp>
+    <kd>100.0</kd>
+    <minDepth>0.001</minDepth>
   </gazebo>
   <gazebo reference="right_wheel_link">
-    <mu1>1.0</mu1>
-    <mu2>1.0</mu2>
-    <kp>1e5</kp>
-    <kd>1.0</kd>
+    <selfCollide>false</selfCollide>
+    <mu1>1.2</mu1>
+    <mu2>1.2</mu2>
+    <kp>1e4</kp>
+    <kd>100.0</kd>
+    <minDepth>0.001</minDepth>
+  </gazebo>
+  <gazebo reference="front_left_fixed_wheel_link">
+    <selfCollide>false</selfCollide>
+    <mu1>0.8</mu1>
+    <mu2>0.8</mu2>
+    <kp>1e4</kp>
+    <kd>50.0</kd>
+  </gazebo>
+  <gazebo reference="front_right_fixed_wheel_link">
+    <selfCollide>false</selfCollide>
+    <mu1>0.8</mu1>
+    <mu2>0.8</mu2>
+    <kp>1e4</kp>
+    <kd>50.0</kd>
+  </gazebo>
+  <gazebo reference="back_left_fixed_wheel_link">
+    <selfCollide>false</selfCollide>
+    <mu1>0.8</mu1>
+    <mu2>0.8</mu2>
+    <kp>1e4</kp>
+    <kd>50.0</kd>
+  </gazebo>
+  <gazebo reference="back_right_fixed_wheel_link">
+    <selfCollide>false</selfCollide>
+    <mu1>0.8</mu1>
+    <mu2>0.8</mu2>
+    <kp>1e4</kp>
+    <kd>50.0</kd>
   </gazebo>
   <ros2_control name="GazeboSystem" type="system">

File: simulation/src/gazebo_robot_had2503_demo/urdf/had2503.urdf (robot description, URDF)
Before this commit: robot HAD2503-D-DEX1, 39 links, 38 joints
Links:
- link ankle_pitch_link: geometry collision box size=0.099712 0.240379 0.308274; visual mesh filename=file:///home/hs/testCode/simulation/install/gazebo_robot_ha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
- link back_left_fixed_wheel_link: geometry collision box size=0.085327 0.057000 0.128182; visual mesh filename=file:///home/hs/testCode/simulation/install/gazebo_robot_ha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
- link back_right_fixed_wheel_link: geometry collision box size=0.085330 0.057000 0.128184; visual mesh filename=file:///home/hs/testCode/simulation/install/gazebo_robot_ha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
- link base_link: geometry collision box size=0.543727 0.541500 0.255026; visual mesh filename=file:///home/hs/testCode/simulation/install/gazebo_robot_ha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
- link front_left_fixed_wheel_link: geometry collision box size=0.085311 0.057000 0.128174; visual mesh filename=file:///home/hs/testCode/simulation/install/gazebo_robot_ha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
- link front_right_fixed_wheel_link: geometry collision box size=0.085345 0.057000 0.128191; visual mesh filename=file:///home/hs/testCode/simulation/install/gazebo_robot_ha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
- link head_pitch_link: geometry collision box size=0.186592 0.169976 0.217884; visual mesh filename=file:///home/hs/testCode/simulation/install/gazebo_robot_ha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
- link head_yaw_link: geometry collision box size=0.094050 0.108300 0.208346; visual mesh filename=file:///home/hs/testCode/simulation/install/gazebo_robot_ha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
- link hip_pitch_link: geometry collision box size=0.119723 0.218500 0.138525; visual mesh filename=file:///home/hs/testCode/simulation/install/gazebo_robot_ha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
- link knee_pitch_link: geometry collision box size=0.116078 0.270987 0.392722; visual mesh filename=file:///home/hs/testCode/simulation/install/gazebo_robot_ha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
- link left_dex1_finger_link_1: geometry collision box size=0.049400 0.057000 0.114000; visual mesh filename=file:///home/hs/testCode/simulation/install/gazebo_robot_ha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
- link left_dex1_finger_link_2: geometry collision box size=0.049400 0.057000 0.114000; visual mesh filename=file:///home/hs/testCode/simulation/install/gazebo_robot_ha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
- link left_elbow_link: geometry collision box size=0.097850 0.075922 0.181687; visual mesh filename=file:///home/hs/testCode/simulation/install/gazebo_robot_ha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
- link left_shoulder_pitch_link: geometry collision box size=0.087875 0.090122 0.076000; visual mesh filename=file:///home/hs/testCode/simulation/install/gazebo_robot_ha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
- link left_shoulder_roll_link: geometry collision box size=0.097850 0.075969 0.164825; visual mesh filename=file:///home/hs/testCode/simulation/install/gazebo_robot_ha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
- link left_shoulder_yaw_link: geometry collision box size=0.087875 0.076000 0.089647; visual mesh filename=file:///home/hs/testCode/simulation/install/gazebo_robot_ha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
- link left_wheel_height_link: geometry collision box size=0.144711 0.122028 0.132017; visual mesh filename=file:///home/hs/testCode/simulation/install/gazebo_robot_ha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
- link left_wheel_link: geometry collision cylinder length=0.038 radius=0.077; visual mesh filename=file:///home/hs/testCode/simulation/install/gazebo_robot_ha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
- link left_wrist_pitch_link: geometry collision box size=0.076950 0.076950 0.104900; visual mesh filename=file:///home/hs/testCode/simulation/install/gazebo_robot_ha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
- link left_wrist_roll_link: geometry collision box size=0.084550 0.070853 0.140071; visual mesh filename=file:///home/hs/testCode/simulation/install/gazebo_robot_ha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
- link left_wrist_yaw_link: geometry collision box size=0.070798 0.084550 0.069350; visual mesh filename=file:///home/hs/testCode/simulation/install/gazebo_robot_ha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
- link right_dex1_finger_link_1: geometry collision box size=0.049400 0.057000 0.114000; visual mesh filename=file:///home/hs/testCode/simulation/install/gazebo_robot_ha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
- link right_dex1_finger_link_2: geometry collision box size=0.049400 0.057000 0.114000; visual mesh filename=file:///home/hs/testCode/simulation/install/gazebo_robot_ha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
- link right_elbow_link: geometry collision box size=0.097850 0.075922 0.181687; visual mesh filename=file:///home/hs/testCode/simulation/install/gazebo_robot_ha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
- link right_shoulder_pitch_link: geometry collision box size=0.087875 0.090122 0.076000; visual mesh filename=file:///home/hs/testCode/simulation/install/gazebo_robot_ha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
- link right_shoulder_roll_link: geometry collision box size=0.097835 0.076056 0.164825; visual mesh filename=file:///home/hs/testCode/simulation/install/gazebo_robot_ha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
- link right_shoulder_yaw_link: geometry collision box size=0.087875 0.076000 0.089647; visual mesh filename=file:///home/hs/testCode/simulation/install/gazebo_robot_ha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
- link right_wheel_height_link: geometry collision box size=0.144870 0.122027 0.131964; visual mesh filename=file:///home/hs/testCode/simulation/install/gazebo_robot_ha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
- link right_wheel_link: geometry collision cylinder length=0.038 radius=0.077; visual mesh filename=file:///home/hs/testCode/simulation/install/gazebo_robot_ha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
- link right_wrist_pitch_link: geometry collision box size=0.076950 0.076950 0.104900; visual mesh filename=file:///home/hs/testCode/simulation/install/gazebo_robot_ha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
- link right_wrist_roll_link: geometry collision box size=0.084550 0.070853 0.140071; visual mesh filename=file:///home/hs/testCode/simulation/install/gazebo_robot_ha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
- link right_wrist_yaw_link: geometry collision box size=0.070798 0.084550 0.069350; visual mesh filename=file:///home/hs/testCode/simulation/install/gazebo_robot_ha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
- link waist_pitch_link: geometry collision box size=0.095000 0.118750 0.181925; visual mesh filename=file:///home/hs/testCode/simulation/install/gazebo_robot_ha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
- link waist_roll_link: geometry collision box size=0.210955 0.305231 0.373981; visual mesh filename=file:///home/hs/testCode/simulation/install/gazebo_robot_ha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
- link waist_yaw_link: geometry collision box size=0.094992 0.098800 0.106398; visual mesh filename=file:///home/hs/testCode/simulation/install/gazebo_robot_ha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

File: simulation/src/gazebo_robot_had2503_demo/urdf/had2503_links.urdf.xacro (robot description, xacro)
@@ -36,9 +36,8 @@
     <collision>
       <origin
-        xyz="0 0 0"
-        rpy="0 0 0" />
-      <geometry>
-        <mesh
-          filename="file://$(find gazebo_robot_had2503_demo)/meshes/base_link.STL" />
+        xyz="0.000000 0.000000 0.118724"
+        rpy="0 0 0" />
+      <geometry>
+        <box size="0.543727 0.541500 0.255026" />
       </geometry>
     </collision>
@@ -76,9 +75,8 @@
     <collision>
       <origin
-        xyz="0 0 0"
-        rpy="0 0 0" />
-      <geometry>
-        <mesh
-          filename="file://$(find gazebo_robot_had2503_demo)/meshes/front_left_fixed_wheel_link.STL" />
+        xyz="-0.009962 0.000000 -0.067460"
+        rpy="0 0 0" />
+      <geometry>
+        <box size="0.085311 0.057000 0.128174" />
       </geometry>
     </collision>
@@ -129,9 +127,8 @@
     <collision>
       <origin
-        xyz="0 0 0"
-        rpy="0 0 0" />
-      <geometry>
-        <mesh
-          filename="file://$(find gazebo_robot_had2503_demo)/meshes/front_right_fixed_wheel_link.STL" />
+        xyz="-0.009996 0.000000 -0.067469"
+        rpy="0 0 0" />
+      <geometry>
+        <box size="0.085345 0.057000 0.128191" />
       </geometry>
     </collision>
@@ -182,9 +179,8 @@
     <collision>
       <origin
-        xyz="0 0 0"
-        rpy="0 0 0" />
-      <geometry>
-        <mesh
-          filename="file://$(find gazebo_robot_had2503_demo)/meshes/back_left_fixed_wheel_link.STL" />
+        xyz="-0.010028 0.000000 -0.067464"
+        rpy="0 0 0" />
+      <geometry>
+        <box size="0.085327 0.057000 0.128182" />
       </geometry>
     </collision>
@@ -235,9 +231,8 @@
     <collision>
       <origin
-        xyz="0 0 0"
-        rpy="0 0 0" />
-      <geometry>
-        <mesh
-          filename="file://$(find gazebo_robot_had2503_demo)/meshes/back_right_fixed_wheel_link.STL" />
+        xyz="-0.009974 0.000000 -0.067465"
+        rpy="0 0 0" />
+      <geometry>
+        <box size="0.085330 0.057000 0.128184" />
       </geometry>
     </collision>
@@ -288,9 +283,8 @@
     <collision>
       <origin
-        xyz="0 0 0"
-        rpy="0 0 0" />
-      <geometry>
-        <mesh
-          filename="file://$(find gazebo_robot_had2503_demo)/meshes/ankle_pitch_link.STL" />
+        xyz="-0.000009 -0.000000 0.113251"
+        rpy="0 0 0" />
+      <geometry>
+        <box size="0.099712 0.240379 0.308274" />
       </geometry>
     </collision>
@@ -346,9 +340,8 @@
     <collision>
       <origin
-        xyz="0 0 0"
-        rpy="0 0 0" />
-      <geometry>
-        <mesh
-          filename="file://$(find gazebo_robot_had2503_demo)/meshes/knee_pitch_link.STL" />
+        xyz="-0.002268 0.000000 0.154196"
+        rpy="0 0 0" />
+      <geometry>
+        <box size="0.116078 0.270987 0.392722" />
       </geometry>
     </collision>
@@ -404,9 +397,8 @@
     <collision>
       <origin
-        xyz="0 0 0"
-        rpy="0 0 0" />
-      <geometry>
-        <mesh
-          filename="file://$(find gazebo_robot_had2503_demo)/meshes/hip_pitch_link.STL" />
+        xyz="-0.003681 0.000000 0.019587"
+        rpy="0 0 0" />
+      <geometry>
+        <box size="0.119723 0.218500 0.138525" />
       </geometry>
     </collision>
@@ -462,9 +454,8 @@
     <collision>
       <origin
-        xyz="0 0 0"
-        rpy="0 0 0" />
-      <geometry>
-        <mesh
-          filename="file://$(find gazebo_robot_had2503_demo)/meshes/waist_yaw_link.STL" />
+        xyz="0.000000 -0.002000 0.092499"
+        rpy="0 0 0" />
+      <geometry>
+        <box size="0.094992 0.098800 0.106398" />
       </geometry>
     </collision>
@@ -520,9 +511,8 @@
     <collision>
       <origin
-        xyz="0 0 0"
-        rpy="0 0 0" />
-      <geometry>
-        <mesh
-          filename="file://$(find gazebo_robot_had2503_demo)/meshes/waist_pitch_link.STL" />
+        xyz="-0.000000 0.000000 0.045750"
+        rpy="0 0 0" />
+      <geometry>
+        <box size="0.095000 0.118750 0.181925" />
       </geometry>
     </collision>
@@ -578,9 +568,8 @@
     <collision>
       <origin
-        xyz="0 0 0"
-        rpy="0 0 0" />
-      <geometry>
-        <mesh
-          filename="file://$(find gazebo_robot_had2503_demo)/meshes/waist_roll_link.STL" />
+        xyz="-0.023473 0.000000 0.140421"
+        rpy="0 0 0" />
+      <geometry>
+        <box size="0.210955 0.305231 0.373981" />
       </geometry>
     </collision>
@@ -636,9 +625,8 @@
     <collision>
       <origin
-        xyz="0 0 0"
-        rpy="0 0 0" />
-      <geometry>
-        <mesh
-          filename="file://$(find gazebo_robot_had2503_demo)/meshes/right_shoulder_pitch_link.STL" />
+        xyz="-0.002750 -0.095433 0.000000"
+        rpy="0 0 0" />
+      <geometry>
+        <box size="0.087875 0.090122 0.076000" />
       </geometry>
     </collision>
@@ -694,9 +682,8 @@
     <collision>
       <origin
-        xyz="0 0 0"
-        rpy="0 0 0" />
-      <geometry>
-        <mesh
-          filename="file://$(find gazebo_robot_had2503_demo)/meshes/right_shoulder_roll_link.STL" />
+        xyz="0.000008 0.000062 -0.046750"
+        rpy="0 0 0" />
+      <geometry>
+        <box size="0.097835 0.076056 0.164825" />
       </geometry>
     </collision>
@@ -752,9 +739,8 @@
     <collision>
       <origin
-        xyz="0 0 0"
-        rpy="0 0 0" />
-      <geometry>
-        <mesh
-          filename="file://$(find gazebo_robot_had2503_demo)/meshes/right_shoulder_yaw_link.STL" />
+        xyz="0.002750 0.000000 -0.119683"
+        rpy="0 0 0" />
+      <geometry>
+        <box size="0.087875 0.076000 0.089647" />
       </geometry>
     </collision>
@@ -810,9 +796,8 @@
     <collision>
       <origin
-        xyz="0 0 0"
-        rpy="0 0 0" />
-      <geometry>
-        <mesh
-          filename="file://$(find gazebo_robot_had2503_demo)/meshes/right_elbow_link.STL" />
+        xyz="0.000000 -0.000012 -0.055625"
+        rpy="0 0 0" />
+      <geometry>
+        <box size="0.097850 0.075922 0.181687" />
       </geometry>
     </collision>
@@ -868,9 +853,8 @@
     <collision>
       <origin
-        xyz="0 0 0"
-        rpy="0 0 0" />
-      <geometry>
-        <mesh
-          filename="file://$(find gazebo_robot_had2503_demo)/meshes/right_wrist_yaw_link.STL" />
+        xyz="0.000000 0.000000 -0.098200"
+        rpy="0 0 0" />
+      <geometry>
+        <box size="0.070798 0.084550 0.069350" />
       </geometry>
     </collision>
@@ -926,9 +910,8 @@
     <collision>
       <origin
-        xyz="0 0 0"
-        rpy="0 0 0" />
-      <geometry>
-        <mesh
-          filename="file://$(find gazebo_robot_had2503_demo)/meshes/right_wrist_pitch_link.STL" />
+        xyz="0.003250 -0.003000 -0.026272"
+        rpy="0 0 0" />
+      <geometry>
+        <box size="0.076950 0.076950 0.104900" />
       </geometry>
     </collision>
@@ -984,9 +967,8 @@
     <collision>
       <origin
-        xyz="0 0 0"
-        rpy="0 0 0" />
-      <geometry>
-        <mesh
-          filename="file://$(find gazebo_robot_had2503_demo)/meshes/right_wrist_roll_link.STL" />
+        xyz="0.000000 0.000000 -0.044779"
+        rpy="0 0 0" />
+      <geometry>
+        <box size="0.084550 0.070853 0.140071" />
       </geometry>
     </collision>
@@ -1042,9 +1024,8 @@
     <collision>
       <origin
-        xyz="0 0 0"
-        rpy="0 0 0" />
-      <geometry>
-        <mesh
-          filename="file://$(find gazebo_robot_had2503_demo)/meshes/right_dex1_finger_link_1.STL" />
+        xyz="0.006000 -0.015000 -0.055000"
+        rpy="0 0 0" />
+      <geometry>
+        <box size="0.049400 0.057000 0.114000" />
       </geometry>
     </collision>
@@ -1100,9 +1081,8 @@
     <collision>
       <origin
-        xyz="0 0 0"
-        rpy="0 0 0" />
-      <geometry>
-        <mesh
-          filename="file://$(find gazebo_robot_had2503_demo)/meshes/right_dex1_finger_link_2.STL" />
+        xyz="-0.011000 0.015000 -0.055000"
+        rpy="0 0 0" />
+      <geometry>
+        <box size="0.049400 0.057000 0.114000" />
       </geometry>
     </collision>
@@ -1158,9 +1138,8 @@
     <collision>
       <origin
-        xyz="0 0 0"
-        rpy="0 0 0" />
-      <geometry>
-        <mesh
-          filename="file://$(find gazebo_robot_had2503_demo)/meshes/left_shoulder_pitch_link.STL" />
+        xyz="-0.002750 0.095433 0.000000"
+        rpy="0 0 0" />
+      <geometry>
+        <box size="0.087875 0.090122 0.076000" />
       </geometry>
     </collision>
@@ -1216,9 +1195,8 @@
     <collision>
       <origin
-        xyz="0 0 0"
-        rpy="0 0 0" />
-      <geometry>
-        <mesh
-          filename="file://$(find gazebo_robot_had2503_demo)/meshes/left_shoulder_roll_link.STL" />
+        xyz="0.000000 -0.000016 -0.046750"
+        rpy="0 0 0" />
+      <geometry>
+        <box size="0.097850 0.075969 0.164825" />
       </geometry>
     </collision>
@@ -1274,9 +1252,8 @@
     <collision>
       <origin
-        xyz="0 0 0"
-        rpy="0 0 0" />
-      <geometry>
-        <mesh
-          filename="file://$(find gazebo_robot_had2503_demo)/meshes/left_shoulder_yaw_link.STL" />
+        xyz="0.002750 0.000000 -0.119683"
+        rpy="0 0 0" />
+      <geometry>
+        <box size="0.087875 0.076000 0.089647" />
       </geometry>
     </collision>
@@ -1332,9 +1309,8 @@
     <collision>
       <origin
-        xyz="0 0 0"
-        rpy="0 0 0" />
-      <geometry>
-        <mesh
-          filename="file://$(find gazebo_robot_had2503_demo)/meshes/left_elbow_link.STL" />
+        xyz="0.000000 0.000012 -0.055625"
+        rpy="0 0 0" />
+      <geometry>
+        <box size="0.097850 0.075922 0.181687" />
       </geometry>
     </collision>
@@ -1390,9 +1366,8 @@
     <collision>
       <origin
-        xyz="0 0 0"
-        rpy="0 0 0" />
-      <geometry>
-        <mesh
-          filename="file://$(find gazebo_robot_had2503_demo)/meshes/left_wrist_yaw_link.STL" />
+        xyz="0.000000 0.000000 -0.098200"
+        rpy="0 0 0" />
+      <geometry>
+        <box size="0.070798 0.084550 0.069350" />
       </geometry>
     </collision>
@@ -1448,9 +1423,8 @@
     <collision>
       <origin
-        xyz="0 0 0"
-        rpy="0 0 0" />
-      <geometry>
-        <mesh
-          filename="file://$(find gazebo_robot_had2503_demo)/meshes/left_wrist_pitch_link.STL" />
+        xyz="0.003250 -0.003250 -0.026272"
+        rpy="0 0 0" />
+      <geometry>
+        <box size="0.076950 0.076950 0.104900" />
       </geometry>
     </collision>
@@ -1506,9 +1480,8 @@
     <collision>
       <origin
-        xyz="0 0 0"
-        rpy="0 0 0" />
-      <geometry>
-        <mesh
-          filename="file://$(find gazebo_robot_had2503_demo)/meshes/left_wrist_roll_link.STL" />
+        xyz="0.000000 0.000000 -0.044779"
+        rpy="0 0 0" />
+      <geometry>
+        <box size="0.084550 0.070853 0.140071" />
       </geometry>
     </collision>
@@ -1564,9 +1537,8 @@
     <collision>
       <origin
-        xyz="0 0 0"
-        rpy="0 0 0" />
-      <geometry>
-        <mesh
-          filename="file://$(find gazebo_robot_had2503_demo)/meshes/left_dex1_finger_link_2.STL" />
+        xyz="-0.011000 0.015000 -0.055000"
+        rpy="0 0 0" />
+      <geometry>
+        <box size="0.049400 0.057000 0.114000" />
       </geometry>
     </collision>
@@ -1622,9 +1594,8 @@
     <collision>
       <origin
-        xyz="0 0 0"
-        rpy="0 0 0" />
-      <geometry>
-        <mesh
-          filename="file://$(find gazebo_robot_had2503_demo)/meshes/left_dex1_finger_link_1.STL" />
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